Commit message: my robot on  Gazebo can't move lol

File: src/robot_description/robot/visual/robot.urdf (robot description, URDF)
Before this commit: robot fake-limo, 8 links, 7 joints
Links:
- removed link font_left_wheel_joint_link
- removed link font_left_wheel_link
- removed link font_right_wheel_joint_link
- removed link font_right_wheel_link
- added link front_left_wheel_joint_link, mass 0.1
- added link front_left_wheel_link, mass 0.1; collision cylinder length=0.01 radius=0.045; visual cylinder length=0.01 radius=0.045
- added link front_right_wheel_joint_link, mass 0.1
- added link front_right_wheel_link, mass 0.1; collision cylinder length=0.01 radius=0.045; visual cylinder length=0.01 radius=0.045
Joints:
- removed joint font_left_wheel
- removed joint font_left_wheel_joint
- removed joint font_right_wheel
- removed joint font_right_wheel_joint
- added joint front_left_wheel: type continuous, parent front_left_wheel_joint_link, child front_left_wheel_link, origin xyz=0.0 0.0 0.0 rpy=-1.57 0.0 0.0, axis 0.0 0.0 1.0, limit lower=0.0 upper=0.0 effort=0.0 velocity=0.0
- added joint front_left_wheel_joint: type revolute, parent base_link, child front_left_wheel_joint_link, origin xyz=0.10 0.07 0.045 rpy=0.0 0.0 0.0, axis 0.0 0.0 1.0, limit lower=-1.57 upper=1.57 effort=0.0 velocity=0.0
- added joint front_right_wheel: type continuous, parent front_right_wheel_joint_link, child front_right_wheel_link, origin xyz=0.0 0.0 0.0 rpy=-1.57 0.0 0.0, axis 0.0 0.0 1.0, limit lower=0.0 upper=0.0 effort=0.0 velocity=0.0
- added joint front_right_wheel_joint: type revolute, parent base_link, child front_right_wheel_joint_link, origin xyz=0.10 -0.07 0.045 rpy=0.0 0.0 0.0, axis 0.0 0.0 1.0, limit lower=-1.57 upper=1.57 effort=0.0 velocity=0.0

Commit message: Update joint limits for front wheel joints in URDF

File: src/robot_description/robot/visual/robot.urdf (robot description, URDF)
Before this commit: robot fake-limo, 8 links, 7 joints
Joints:
- joint front_left_wheel_joint: limit lower=-1.57 upper=1.57 effort=0.0 velocity=0.0 -> lower=-0.7854 upper=0.7854 effort=0.0 velocity=0.0
- joint front_right_wheel_joint: limit lower=-1.57 upper=1.57 effort=0.0 velocity=0.0 -> lower=-0.7854 upper=0.7854 effort=0.0 velocity=0.0

Commit message: Try to add stl on my world and yes!!! BUG.

File: src/robot_description/robot/visual/robot.urdf (robot description, URDF)
Before this commit: robot fake-limo, 8 links, 7 joints
Links:
- link base_link: mass 1.0 -> 0.0
