Commit message: Update mesh scale values in URDF for consistency

File: src/robot_description/robot/visual/robot.urdf.xacro (robot description, xacro)
@@ -24,5 +24,5 @@
             <origin xyz="0.0 0.0 0.0" rpy="0.0 0.0 0.0"/>
             <geometry>
-                <mesh filename="package://robot_description/meshes/limo_base.stl" scale="1 1 1"/>
+                <mesh filename="package://robot_description/meshes/limo_base.stl" scale="1.0"/>
             </geometry>
             <material name="">
@@ -33,5 +33,5 @@
             <origin xyz="0.0 0.0 0.0" rpy="0.0 0.0 0.0"/>
             <geometry>
-                <mesh filename="package://robot_description/meshes/limo_base.stl" scale="1 1 1"/>
+                <mesh filename="package://robot_description/meshes/limo_base.stl" scale="1.0"/>
             </geometry>
         </collision>
@@ -68,5 +68,5 @@
             <origin xyz="0.0 0.0 0.0" rpy="0.0 0.0 0.0"/>
             <geometry>
-                <mesh filename="package://robot_description/meshes/limo_wheel.stl" scale="1 1 1"/>
+                <mesh filename="package://robot_description/meshes/limo_wheel.stl" scale="1.0"/>
             </geometry>
             <material name="">
@@ -77,5 +77,5 @@
             <origin xyz="0.0 0.0 0.0" rpy="0.0 0.0 0.0"/>
             <geometry>
-                <mesh filename="package://robot_description/meshes/limo_wheel.stl" scale="1 1 1"/>
+                <mesh filename="package://robot_description/meshes/limo_wheel.stl" scale="1.0"/>
             </geometry>
         </collision>
@@ -112,5 +112,5 @@
             <origin xyz="0.0 0.0 0.0" rpy="0.0 0.0 0.0"/>
             <geometry>
-                <mesh filename="package://robot_description/meshes/limo_wheel.stl" scale="1 1 1"/>
+                <mesh filename="package://robot_description/meshes/limo_wheel.stl" scale="1.0"/>
             </geometry>
             <material name="">
@@ -121,5 +121,5 @@
             <origin xyz="0.0 0.0 0.0" rpy="0.0 0.0 0.0"/>
             <geometry>
-                <mesh filename="package://robot_description/meshes/limo_wheel.stl" scale="1 1 1"/>
+                <mesh filename="package://robot_description/meshes/limo_wheel.stl" scale="1.0"/>
             </geometry>
         </collision>
@@ -142,5 +142,5 @@
             <origin xyz="0.0 0.0 0.0" rpy="0.0 0.0 0.0"/>
             <geometry>
-                <mesh filename="package://robot_description/meshes/limo_wheel.stl" scale="1 1 1"/>
+                <mesh filename="package://robot_description/meshes/limo_wheel.stl" scale="1.0"/>
             </geometry>
             <material name="">
@@ -151,5 +151,5 @@
             <origin xyz="0.0 0.0 0.0" rpy="0.0 0.0 0.0"/>
             <geometry>
-                <mesh filename="package://robot_description/meshes/limo_wheel.stl" scale="1 1 1"/>
+                <mesh filename="package://robot_description/meshes/limo_wheel.stl" scale="1.0"/>
             </geometry>
         </collision>
@@ -172,5 +172,5 @@
             <origin xyz="0.0 0.0 0.0" rpy="0.0 0.0 0.0"/>
             <geometry>
-                <mesh filename="package://robot_description/meshes/limo_wheel.stl" scale="1 1 1"/>
+                <mesh filename="package://robot_description/meshes/limo_wheel.stl" scale="1.0"/>
             </geometry>
             <material name="">
@@ -181,5 +181,5 @@
             <origin xyz="0.0 0.0 0.0" rpy="0.0 0.0 0.0"/>
             <geometry>
-                <mesh filename="package://robot_description/meshes/limo_wheel.stl" scale="1 1 1"/>
+                <mesh filename="package://robot_description/meshes/limo_wheel.stl" scale="1.0"/>
             </geometry>
         </collision>
