Commit message: add Gazebo_control but not test

File: src/robot_description/description/robot_core.urdf.xacro (robot description, xacro)
@@ -1,6 +1,18 @@
 <?xml version="1.0"?>
-<robot name="fake-limo">
+<robot xmlns:xacro="http://www.ros.org/wiki/xacro">
+    <!-- Import the inertial macros -->
+    <xacro:include filename="inertial_macros.xacro"/>
+    <!-- COLOR NAME  -->
+    <material name="white">
+        <color rgba="1 1 1 1" />
+    </material>
+    <material name="black">
+        <color rgba="0 0 0 1"/>
+    </material>
+     <material name="blue">
+        <color rgba="0 0 1 1"/>
+    </material>
     <!-- base link -->
-    <link name="base_link">
+    <!-- <link name="base_link">
         <inertial>
             <origin xyz="0.0 0.0 0.0" rpy="0.0 0.0 0.0"/>
@@ -8,5 +20,6 @@
             <inertia ixx="0.1" ixy="0.0" ixz="0.0" iyy="0.1" iyz="0.0" izz="0.1"/>
         </inertial>
-    </link>
+    </link> -->
+    <link name="base_link"/>
     <!-- chassis link -->
     <joint name="chassis_joint" type="fixed">
@@ -16,25 +29,29 @@
     </joint>
     <link name="chassis">
-        <inertial>
+        <!-- <inertial>
             <origin xyz="0.0 0.0 0.0" rpy="0.0 0.0 0.0"/>
             <mass value="3.0"/>
             <inertia ixx="0.1" ixy="0.0" ixz="0.0" iyy="0.1" iyz="0.0" izz="0.1"/>
-        </inertial>
-        <visual name="">
-            <origin xyz="0.0 0.0 0.0" rpy="0.0 0.0 0.0"/>
-            <geometry>
-                <mesh filename="package://robot_description/meshes/limo_base.stl" scale="1.0"/>
-            </geometry>
-            <material name="">
-                <color rgba="1.0 1.0 1.0 1.0"/>
-            </material>
-        </visual>
-        <collision>
-            <origin xyz="0.0 0.0 0.0" rpy="0.0 0.0 0.0"/>
-            <geometry>
-                <mesh filename="package://robot_description/meshes/limo_base.stl" scale="1.0"/>
-            </geometry>
-        </collision>
-    </link>
+        </inertial> -->
+        <visual name="">
+            <origin xyz="0.0 0.0 0.0" rpy="0.0 0.0 0.0"/>
+            <geometry>
+                <box size="0.13 0.20 0.1"/>
+            </geometry>
+            <material name="white"/>
+        </visual>
+        <collision>
+            <origin xyz="0.0 0.0 0.0" rpy="0.0 0.0 0.0"/>
+            <geometry>
+                <box size="0.13 0.20 0.1"/>
+            </geometry>
+        </collision>
+        <xacro:inertial_box mass="3.0" x="0.13" y="0.2" z="0.1">
+            <origin xyz="0.0 0.0 0.0" rpy="0 0 0"/>
+        </xacro:inertial_box>
+    </link>
+    <gazebo reference="chassis">
+        <material>Gazebo/White</material>
+    </gazebo>
     <!-- front left wheel -->
     <joint name="front_left_wheel_joint" type="revolute">
@@ -46,9 +63,9 @@
     </joint>
     <link name="front_left_wheel_joint_link">
-        <inertial>
-            <origin xyz="0.0 0.0 0.0" rpy="0.0 0.0 0.0"/>
-            <mass value="0.1"/>
-            <inertia ixx="0.01" ixy="0.0" ixz="0.0" iyy="0.01" iyz="0.0" izz="0.01"/>
-        </inertial>
+        <!-- <inertial>
+            <origin xyz="0.0 0.0 0.0" rpy="0.0 0.0 0.0"/>
+            <mass value="0.1"/>
+            <inertia ixx="0.01" ixy="0.0" ixz="0.0" iyy="0.01" iyz="0.0" izz="0.01"/>
+        </inertial> -->
     </link>
     <joint name="front_left_wheel" type="continuous">
@@ -57,28 +74,32 @@
         <child link="front_left_wheel_link"/>
         <axis xyz="0.0 0.0 1.0"/>
-        <limit lower="0.0" upper="0.0" effort="0.0" velocity="0.0"/>
+        <!-- <limit lower="0.0" upper="0.0" effort="0.0" velocity="0.0"/> -->
     </joint>
     <link name="front_left_wheel_link">
-        <inertial>
-            <origin xyz="0.0 0.0 0.0" rpy="0.0 0.0 0.0"/>
-            <mass value="0.1"/>
-            <inertia ixx="0.01" ixy="0.0" ixz="0.0" iyy="0.01" iyz="0.0" izz="0.01"/>
-        </inertial>
-        <visual name="">
-            <origin xyz="0.0 0.0 0.0" rpy="0.0 0.0 0.0"/>
-            <geometry>
-                <mesh filename="package://robot_description/meshes/limo_wheel.stl" scale="1.0"/>
-            </geometry>
-            <material name="">
-                <color rgba="0.0 0.0 0.0 1.0"/>
-            </material>
-        </visual>
-        <collision>
-            <origin xyz="0.0 0.0 0.0" rpy="0.0 0.0 0.0"/>
-            <geometry>
-                <mesh filename="package://robot_description/meshes/limo_wheel.stl" scale="1.0"/>
-            </geometry>
-        </collision>
-    </link>
+        <!-- <inertial>
+            <origin xyz="0.0 0.0 0.0" rpy="0.0 0.0 0.0"/>
+            <mass value="0.1"/>
+            <inertia ixx="0.01" ixy="0.0" ixz="0.0" iyy="0.01" iyz="0.0" izz="0.01"/>
+        </inertial> -->
+        <visual name="">
+            <origin xyz="0.0 0.0 0.0" rpy="0.0 0.0 0.0"/>
+            <geometry>
+                <cylinder radius="0.045" length="0.01"/>
+            </geometry>
+            <material name="blue"/>
+        </visual>
+        <collision>
+            <origin xyz="0.0 0.0 0.0" rpy="0.0 0.0 0.0"/>
+            <geometry>
+                 <cylinder radius="0.045" length="0.01"/>
+            </geometry>
+        </collision>
+        <xacro:inertial_cylinder mass="0.1" length="0.01" radius="0.045">
+            <origin xyz="0 0 0" rpy="0 0 0"/>
+        </xacro:inertial_cylinder>
+    </link>
+    <gazebo reference="front_left_wheel_link">
+        <material>Gazebo/Blue</material>
+    </gazebo>
     <!-- front right wheel -->
     <joint name="front_right_wheel_joint" type="revolute">
@@ -90,9 +111,9 @@
     </joint>
     <link name="front_right_wheel_joint_link">
-        <inertial>
-            <origin xyz="0.0 0.0 0.0" rpy="0.0 0.0 0.0"/>
-            <mass value="0.1"/>
-            <inertia ixx="0.01" ixy="0.0" ixz="0.0" iyy="0.01" iyz="0.0" izz="0.01"/>
-        </inertial>
+        <!-- <inertial>
+            <origin xyz="0.0 0.0 0.0" rpy="0.0 0.0 0.0"/>
+            <mass value="0.1"/>
+            <inertia ixx="0.01" ixy="0.0" ixz="0.0" iyy="0.01" iyz="0.0" izz="0.01"/>
+        </inertial> -->
     </link>
     <joint name="front_right_wheel" type="continuous">
@@ -101,28 +122,32 @@
         <child link="front_right_wheel_link"/>
         <axis xyz="0.0 0.0 1.0"/>
-        <limit lower="0.0" upper="0.0" effort="0.0" velocity="0.0"/>
+        <!-- <limit lower="0.0" upper="0.0" effort="0.0" velocity="0.0"/> -->
     </joint>
     <link name="front_right_wheel_link">
-        <inertial>
-            <origin xyz="0.0 0.0 0.0" rpy="0.0 0.0 0.0"/>
-            <mass value="0.1"/>
-            <inertia ixx="0.01" ixy="0.0" ixz="0.0" iyy="0.01" iyz="0.0" izz="0.01"/>
-        </inertial>
-        <visual name="">
-            <origin xyz="0.0 0.0 0.0" rpy="0.0 0.0 0.0"/>
-            <geometry>
-                <mesh filename="package://robot_description/meshes/limo_wheel.stl" scale="1.0"/>
-            </geometry>
-            <material name="">
-                <color rgba="0.0 0.0 0.0 1.0"/>
-            </material>
-        </visual>
-        <collision>
-            <origin xyz="0.0 0.0 0.0" rpy="0.0 0.0 0.0"/>
-            <geometry>
-                <mesh filename="package://robot_description/meshes/limo_wheel.stl" scale="1.0"/>
-            </geometry>
-        </collision>
-    </link>
+        <!-- <inertial>
+            <origin xyz="0.0 0.0 0.0" rpy="0.0 0.0 0.0"/>
+            <mass value="0.1"/>
+            <inertia ixx="0.01" ixy="0.0" ixz="0.0" iyy="0.01" iyz="0.0" izz="0.01"/>
+        </inertial> -->
+        <visual name="">
+            <origin xyz="0.0 0.0 0.0" rpy="0.0 0.0 0.0"/>
+            <geometry>
+                <cylinder radius="0.045" length="0.01"/>
+            </geometry>
+            <material name="blue"/>
+        </visual>
+        <collision>
+            <origin xyz="0.0 0.0 0.0" rpy="0.0 0.0 0.0"/>
+            <geometry>
+                 <cylinder radius="0.045" length="0.01"/>
+            </geometry>
+        </collision>
+        <xacro:inertial_cylinder mass="0.1" length="0.01" radius="0.045">
+            <origin xyz="0 0 0" rpy="0 0 0"/>
+        </xacro:inertial_cylinder>
+    </link>
+    <gazebo reference="front_right_wheel_link">
+        <material>Gazebo/Blue</material>
+    </gazebo>
     <!-- back left wheel -->
     <joint name="back_left_wheel" type="continuous">
@@ -131,28 +156,32 @@
         <child link="back_left_wheel_link"/>
         <axis xyz="0.0 0.0 1.0"/>
-        <limit lower="0.0" upper="0.0" effort="0.0" velocity="0.0"/>
+        <!-- <limit lower="0.0" upper="0.0" effort="0.0" velocity="0.0"/> -->
     </joint>
     <link name="back_left_wheel_link">
-        <inertial>
-            <origin xyz="0.0 0.0 0.0" rpy="0.0 0.0 0.0"/>
-            <mass value="0.1"/>
-            <inertia ixx="0.01" ixy="0.0" ixz="0.0" iyy="0.01" iyz="0.0" izz="0.01"/>
-        </inertial>
-        <visual name="">
-            <origin xyz="0.0 0.0 0.0" rpy="0.0 0.0 0.0"/>
-            <geometry>
-                <mesh filename="package://robot_description/meshes/limo_wheel.stl" scale="1.0"/>
-            </geometry>
-            <material name="">
-                <color rgba="0.0 0.0 0.0 1.0"/>
-            </material>
-        </visual>
-        <collision>
-            <origin xyz="0.0 0.0 0.0" rpy="0.0 0.0 0.0"/>
-            <geometry>
-                <mesh filename="package://robot_description/meshes/limo_wheel.stl" scale="1.0"/>
-            </geometry>
-        </collision>
-    </link>
+        <!-- <inertial>
+            <origin xyz="0.0 0.0 0.0" rpy="0.0 0.0 0.0"/>
+            <mass value="0.1"/>
+            <inertia ixx="0.01" ixy="0.0" ixz="0.0" iyy="0.01" iyz="0.0" izz="0.01"/>
+        </inertial> -->
+        <visual name="">
+            <origin xyz="0.0 0.0 0.0" rpy="0.0 0.0 0.0"/>
+            <geometry>
+                <cylinder radius="0.045" length="0.01"/>
+            </geometry>
+            <material name="black"/>
+        </visual>
+        <collision>
+            <origin xyz="0.0 0.0 0.0" rpy="0.0 0.0 0.0"/>
+            <geometry>
+                 <cylinder radius="0.045" length="0.01"/>
+            </geometry>
+        </collision>
+        <xacro:inertial_cylinder mass="0.1" length="0.01" radius="0.045">
+            <origin xyz="0 0 0" rpy="0 0 0"/>
+        </xacro:inertial_cylinder>
+    </link>
+    <gazebo reference="back_left_wheel_link">
+        <material>Gazebo/Black</material>
+    </gazebo>
     <!-- back right wheel -->
     <joint name="back_right_wheel" type="continuous">
@@ -164,50 +193,32 @@
     </joint>
     <link name="back_right_wheel_link">
-        <inertial>
-            <origin xyz="0.0 0.0 0.0" rpy="0.0 0.0 0.0"/>
-            <mass value="0.1"/>
-            <inertia ixx="0.01" ixy="0.0" ixz="0.0" iyy="0.01" iyz="0.0" izz="0.01"/>
-        </inertial>
-        <visual name="">
-            <origin xyz="0.0 0.0 0.0" rpy="0.0 0.0 0.0"/>
-            <geometry>
-                <mesh filename="package://robot_description/meshes/limo_wheel.stl" scale="1.0"/>
-            </geometry>
-            <material name="">
-                <color rgba="0.0 0.0 0.0 1.0"/>
-            </material>
-        </visual>
-        <collision>
-            <origin xyz="0.0 0.0 0.0" rpy="0.0 0.0 0.0"/>
-            <geometry>
-                <mesh filename="package://robot_description/meshes/limo_wheel.stl" scale="1.0"/>
-            </geometry>
-        </collision>
-    </link>
+        <!-- <inertial>
+            <origin xyz="0.0 0.0 0.0" rpy="0.0 0.0 0.0"/>
+            <mass value="0.1"/>
+            <inertia ixx="0.01" ixy="0.0" ixz="0.0" iyy="0.01" iyz="0.0" izz="0.01"/>
+        </inertial> -->
+        <visual name="">
+            <origin xyz="0.0 0.0 0.0" rpy="0.0 0.0 0.0"/>
+            <geometry>
+                <cylinder radius="0.045" length="0.01"/>
+            </geometry>
+            <material name="black"/>
+        </visual>
+        <collision>
+            <origin xyz="0.0 0.0 0.0" rpy="0.0 0.0 0.0"/>
+            <geometry>
+                 <cylinder radius="0.045" length="0.01"/>
+            </geometry>
+        </collision>
+        <xacro:inertial_cylinder mass="0.1" length="0.01" radius="0.045">
+            <origin xyz="0 0 0" rpy="0 0 0"/>
+        </xacro:inertial_cylinder>
+    </link>
+    <gazebo reference="back_left_wheel_link">
+        <material>Gazebo/Black</material>
+    </gazebo>
     <!-- Gazebo specific elements -->
-    <gazebo>
+    <!-- <gazebo>
         <plugin name="gazebo_ros_control" filename="libgazebo_ros_control.so"/>
-    </gazebo>
-    <!-- ros2 contoller -->
-    <ros2_control name="fake_limo_control" type="system">
-        <hardware>
-            <plugin>gazebo_ros2_control/GazeboSystem</plugin>
-        </hardware>
-        <joint name="front_left_wheel">
-            <command_interface name="velocity"/>
-            <state_interface name="velocity"/>
-        </joint>
-        <joint name="front_right_wheel">
-            <command_interface name="velocity"/>
-            <state_interface name="velocity"/>
-        </joint>
-        <joint name="back_left_wheel">
-            <command_interface name="velocity"/>
-            <state_interface name="velocity"/>
-        </joint>
-        <joint name="back_right_wheel">
-            <command_interface name="velocity"/>
-            <state_interface name="velocity"/>
-        </joint>
-    </ros2_control>
+    </gazebo> -->
 </robot>

Commit message: Change InvertKinematic round 1

File: src/robot_description/description/robot_core.urdf.xacro (robot description, xacro)
@@ -16,5 +16,5 @@
     <!-- chassis link -->
     <joint name="chassis_joint" type="fixed">
-        <origin xyz="0.0 0.0 0.095" rpy="0.0 0.0 1.57"/>
+        <origin xyz="0.0 0.0 0.095" rpy="0.0 0.0 0.0"/>
         <parent link="base_link"/>
         <child link="chassis"/>
@@ -24,5 +24,5 @@
             <origin xyz="0.0 0.0 0.0" rpy="0.0 0.0 0.0"/>
             <geometry>
-                <box size="0.13 0.20 0.1"/>
+                <box size="0.20 0.13 0.1"/>
             </geometry>
             <material name="white"/>
@@ -31,5 +31,5 @@
             <origin xyz="0.0 0.0 0.0" rpy="0.0 0.0 0.0"/>
             <geometry>
-                <box size="0.13 0.20 0.1"/>
+                <box size="0.20 0.13 0.1"/>
             </geometry>
         </collision>
@@ -50,6 +50,6 @@
     </link>
     <joint name="front_left_steering_joint" type="revolute">
-        <origin xyz="0.10 0.07 0.045" rpy="0.0 0.0 0.0"/>
-        <parent link="base_link"/>
+        <origin xyz="0.10 0.07 -0.045" rpy="0.0 0.0 0.0"/>
+        <parent link="chassis"/>
         <child link="front_left_wheel_joint_link"/>
         <axis xyz="0.0 0.0 1.0"/>
@@ -98,6 +98,6 @@
     </link>
     <joint name="front_right_steering_joint" type="revolute">
-        <origin xyz="0.10 -0.07 0.045" rpy="0.0 0.0 0.0"/>
-        <parent link="base_link"/>
+        <origin xyz="0.10 -0.07 -0.045" rpy="0.0 0.0 0.0"/>
+        <parent link="chassis"/>
         <child link="front_right_wheel_joint_link"/>
         <axis xyz="0.0 0.0 1.0"/>
@@ -139,6 +139,6 @@
     <!-- back left wheel -->
     <joint name="back_left_wheel" type="continuous">
-        <origin xyz="-0.10 0.07 0.045" rpy="-1.57 0.0 0.0"/>
-        <parent link="base_link"/>
+        <origin xyz="-0.10 0.07 -0.045" rpy="-1.57 0.0 0.0"/>
+        <parent link="chassis"/>
         <child link="back_left_wheel_link"/>
         <axis xyz="0.0 0.0 1.0"/>
@@ -172,6 +172,6 @@
     <!-- back right wheel -->
     <joint name="back_right_wheel" type="continuous">
-        <origin xyz="-0.10 -0.07 0.045" rpy="-1.57 0.0 0.0"/>
-        <parent link="base_link"/>
+        <origin xyz="-0.10 -0.07 -0.045" rpy="-1.57 0.0 0.0"/>
+        <parent link="chassis"/>
         <child link="back_right_wheel_link"/>
         <axis xyz="0.0 0.0 1.0"/>
