Commit message: Add Sensor to models

File: src/robot_description/description/robot-main.xacro (robot description, xacro)
@@ -3,6 +3,6 @@
     <xacro:include filename="robot_core.urdf.xacro"/>
     <xacro:include filename="gazebo_control.xacro"/>
-    <!-- <xacro:include filename="camera.xacro"/> -->
-    <!-- <xacro:include filename="lidar.xacro"/> -->
-    <!-- <xacro:include filename="imu.xacro"/> -->
+    <xacro:include filename="camera.xacro"/>
+    <xacro:include filename="lidar.xacro"/>
+    <xacro:include filename="imu.xacro"/>
 </robot>

File: src/robot_description/description/robot_core.urdf.xacro (robot description, xacro)
@@ -9,6 +9,9 @@
         <color rgba="0 0 0 1"/>
     </material>
-     <material name="blue">
+    <material name="blue">
         <color rgba="0 0 1 1"/>
+    </material>
+    <material name="red">
+        <color rgba="1 0 0 1"/>
     </material>
     <!-- base link -->
