Commit message: It's Work!!! And yes same has bug

File: src/robot_description/description/gazebo_control.xacro (robot description, xacro)
@@ -3,5 +3,5 @@
     <gazebo>
         <plugin filename="libgazebo_ros2_control.so" name="gazebo_ros2_control">
-            <parameters>$(find robot_controller)/config/example_controllers.yaml</parameters>
+            <parameters>$(find robot_controller)/config/robot_controllers.yaml</parameters>
         </plugin>
     </gazebo>

File: src/robot_description/description/robot_core.urdf.xacro (robot description, xacro)
@@ -14,11 +14,4 @@
     </material>
     <!-- base link -->
-    <!-- <link name="base_link">
-        <inertial>
-            <origin xyz="0.0 0.0 0.0" rpy="0.0 0.0 0.0"/>
-            <mass value="0.0"/>
-            <inertia ixx="0.1" ixy="0.0" ixz="0.0" iyy="0.1" iyz="0.0" izz="0.1"/>
-        </inertial>
-    </link> -->
     <link name="base_link"/>
     <!-- chassis link -->
@@ -29,9 +22,4 @@
     </joint>
     <link name="chassis">
-        <!-- <inertial>
-            <origin xyz="0.0 0.0 0.0" rpy="0.0 0.0 0.0"/>
-            <mass value="3.0"/>
-            <inertia ixx="0.1" ixy="0.0" ixz="0.0" iyy="0.1" iyz="0.0" izz="0.1"/>
-        </inertial> -->
         <visual name="">
             <origin xyz="0.0 0.0 0.0" rpy="0.0 0.0 0.0"/>
@@ -55,5 +43,12 @@
     </gazebo>
     <!-- front left wheel -->
-    <joint name="front_left_wheel_joint" type="revolute">
+    <link name="front_left_wheel_joint_link">
+        <inertial>
+            <origin xyz="0.0 0.0 0.0" rpy="0.0 0.0 0.0"/>
+            <mass value="0.1"/>
+            <inertia ixx="0.01" ixy="0.0" ixz="0.0" iyy="0.01" iyz="0.0" izz="0.01"/>
+        </inertial>
+    </link>
+    <joint name="front_left_wheel_steering_hinge" type="revolute">
         <origin xyz="0.10 0.07 0.045" rpy="0.0 0.0 0.0"/>
         <parent link="base_link"/>
@@ -62,10 +57,26 @@
         <limit lower="-0.7854" upper="0.7854" effort="0.0" velocity="0.0"/>
     </joint>
-    <link name="front_left_wheel_joint_link">
-        <!-- <inertial>
-            <origin xyz="0.0 0.0 0.0" rpy="0.0 0.0 0.0"/>
-            <mass value="0.1"/>
-            <inertia ixx="0.01" ixy="0.0" ixz="0.0" iyy="0.01" iyz="0.0" izz="0.01"/>
-        </inertial> -->
+    <link name="front_left_wheel_link">
+        <inertial>
+            <origin xyz="0.0 0.0 0.0" rpy="0.0 0.0 0.0"/>
+            <mass value="0.1"/>
+            <inertia ixx="0.01" ixy="0.0" ixz="0.0" iyy="0.01" iyz="0.0" izz="0.01"/>
+        </inertial>
+        <visual name="">
+            <origin xyz="0.0 0.0 0.0" rpy="0.0 0.0 0.0"/>
+            <geometry>
+                <cylinder radius="0.045" length="0.01"/>
+            </geometry>
+            <material name="blue"/>
+        </visual>
+        <collision>
+            <origin xyz="0.0 0.0 0.0" rpy="0.0 0.0 0.0"/>
+            <geometry>
+                <cylinder radius="0.045" length="0.01"/>
+            </geometry>
+        </collision>
+        <xacro:inertial_cylinder mass="0.1" length="0.01" radius="0.045">
+            <origin xyz="0 0 0" rpy="0 0 0"/>
+        </xacro:inertial_cylinder>
     </link>
     <joint name="front_left_wheel" type="continuous">
@@ -74,34 +85,17 @@
         <child link="front_left_wheel_link"/>
         <axis xyz="0.0 0.0 1.0"/>
-        <!-- <limit lower="0.0" upper="0.0" effort="0.0" velocity="0.0"/> -->
-    </joint>
-    <link name="front_left_wheel_link">
-        <!-- <inertial>
-            <origin xyz="0.0 0.0 0.0" rpy="0.0 0.0 0.0"/>
-            <mass value="0.1"/>
-            <inertia ixx="0.01" ixy="0.0" ixz="0.0" iyy="0.01" iyz="0.0" izz="0.01"/>
-        </inertial> -->
-        <visual name="">
-            <origin xyz="0.0 0.0 0.0" rpy="0.0 0.0 0.0"/>
-            <geometry>
-                <cylinder radius="0.045" length="0.01"/>
-            </geometry>
-            <material name="blue"/>
-        </visual>
-        <collision>
-            <origin xyz="0.0 0.0 0.0" rpy="0.0 0.0 0.0"/>
-            <geometry>
-                 <cylinder radius="0.045" length="0.01"/>
-            </geometry>
-        </collision>
-        <xacro:inertial_cylinder mass="0.1" length="0.01" radius="0.045">
-            <origin xyz="0 0 0" rpy="0 0 0"/>
-        </xacro:inertial_cylinder>
-    </link>
+    </joint>
     <gazebo reference="front_left_wheel_link">
         <material>Gazebo/Blue</material>
     </gazebo>
     <!-- front right wheel -->
-    <joint name="front_right_wheel_joint" type="revolute">
+    <link name="front_right_wheel_joint_link">
+        <inertial>
+            <origin xyz="0.0 0.0 0.0" rpy="0.0 0.0 0.0"/>
+            <mass value="0.1"/>
+            <inertia ixx="0.01" ixy="0.0" ixz="0.0" iyy="0.01" iyz="0.0" izz="0.01"/>
+        </inertial>
+    </link>
+    <joint name="front_right_wheel_steering_hinge" type="revolute">
         <origin xyz="0.10 -0.07 0.045" rpy="0.0 0.0 0.0"/>
         <parent link="base_link"/>
@@ -110,10 +104,26 @@
         <limit lower="-0.7854" upper="0.7854" effort="0.0" velocity="0.0"/>
     </joint>
-    <link name="front_right_wheel_joint_link">
-        <!-- <inertial>
-            <origin xyz="0.0 0.0 0.0" rpy="0.0 0.0 0.0"/>
-            <mass value="0.1"/>
-            <inertia ixx="0.01" ixy="0.0" ixz="0.0" iyy="0.01" iyz="0.0" izz="0.01"/>
-        </inertial> -->
+    <link name="front_right_wheel_link">
+        <inertial>
+            <origin xyz="0.0 0.0 0.0" rpy="0.0 0.0 0.0"/>
+            <mass value="0.1"/>
+            <inertia ixx="0.01" ixy="0.0" ixz="0.0" iyy="0.01" iyz="0.0" izz="0.01"/>
+        </inertial>
+        <visual name="">
+            <origin xyz="0.0 0.0 0.0" rpy="0.0 0.0 0.0"/>
+            <geometry>
+                <cylinder radius="0.045" length="0.01"/>
+            </geometry>
+            <material name="blue"/>
+        </visual>
+        <collision>
+            <origin xyz="0.0 0.0 0.0" rpy="0.0 0.0 0.0"/>
+            <geometry>
+                <cylinder radius="0.045" length="0.01"/>
+            </geometry>
+        </collision>
+        <xacro:inertial_cylinder mass="0.1" length="0.01" radius="0.045">
+            <origin xyz="0 0 0" rpy="0 0 0"/>
+        </xacro:inertial_cylinder>
     </link>
     <joint name="front_right_wheel" type="continuous">
@@ -122,29 +132,5 @@
         <child link="front_right_wheel_link"/>
         <axis xyz="0.0 0.0 1.0"/>
-        <!-- <limit lower="0.0" upper="0.0" effort="0.0" velocity="0.0"/> -->
-    </joint>
-    <link name="front_right_wheel_link">
-        <!-- <inertial>
-            <origin xyz="0.0 0.0 0.0" rpy="0.0 0.0 0.0"/>
-            <mass value="0.1"/>
-            <inertia ixx="0.01" ixy="0.0" ixz="0.0" iyy="0.01" iyz="0.0" izz="0.01"/>
-        </inertial> -->
-        <visual name="">
-            <origin xyz="0.0 0.0 0.0" rpy="0.0 0.0 0.0"/>
-            <geometry>
-                <cylinder radius="0.045" length="0.01"/>
-            </geometry>
-            <material name="blue"/>
-        </visual>
-        <collision>
-            <origin xyz="0.0 0.0 0.0" rpy="0.0 0.0 0.0"/>
-            <geometry>
-                 <cylinder radius="0.045" length="0.01"/>
-            </geometry>
-        </collision>
-        <xacro:inertial_cylinder mass="0.1" length="0.01" radius="0.045">
-            <origin xyz="0 0 0" rpy="0 0 0"/>
-        </xacro:inertial_cylinder>
-    </link>
+    </joint>
     <gazebo reference="front_right_wheel_link">
         <material>Gazebo/Blue</material>
@@ -156,12 +142,11 @@
         <child link="back_left_wheel_link"/>
         <axis xyz="0.0 0.0 1.0"/>
-        <!-- <limit lower="0.0" upper="0.0" effort="0.0" velocity="0.0"/> -->
     </joint>
     <link name="back_left_wheel_link">
-        <!-- <inertial>
-            <origin xyz="0.0 0.0 0.0" rpy="0.0 0.0 0.0"/>
-            <mass value="0.1"/>
-            <inertia ixx="0.01" ixy="0.0" ixz="0.0" iyy="0.01" iyz="0.0" izz="0.01"/>
-        </inertial> -->
+        <inertial>
+            <origin xyz="0.0 0.0 0.0" rpy="0.0 0.0 0.0"/>
+            <mass value="0.1"/>
+            <inertia ixx="0.01" ixy="0.0" ixz="0.0" iyy="0.01" iyz="0.0" izz="0.01"/>
+        </inertial>
         <visual name="">
             <origin xyz="0.0 0.0 0.0" rpy="0.0 0.0 0.0"/>
@@ -174,5 +159,5 @@
             <origin xyz="0.0 0.0 0.0" rpy="0.0 0.0 0.0"/>
             <geometry>
-                 <cylinder radius="0.045" length="0.01"/>
+                <cylinder radius="0.045" length="0.01"/>
             </geometry>
         </collision>
@@ -193,9 +178,9 @@
     </joint>
     <link name="back_right_wheel_link">
-        <!-- <inertial>
-            <origin xyz="0.0 0.0 0.0" rpy="0.0 0.0 0.0"/>
-            <mass value="0.1"/>
-            <inertia ixx="0.01" ixy="0.0" ixz="0.0" iyy="0.01" iyz="0.0" izz="0.01"/>
-        </inertial> -->
+        <inertial>
+            <origin xyz="0.0 0.0 0.0" rpy="0.0 0.0 0.0"/>
+            <mass value="0.1"/>
+            <inertia ixx="0.01" ixy="0.0" ixz="0.0" iyy="0.01" iyz="0.0" izz="0.01"/>
+        </inertial>
         <visual name="">
             <origin xyz="0.0 0.0 0.0" rpy="0.0 0.0 0.0"/>
@@ -208,17 +193,13 @@
             <origin xyz="0.0 0.0 0.0" rpy="0.0 0.0 0.0"/>
             <geometry>
-                 <cylinder radius="0.045" length="0.01"/>
-            </geometry>
-        </collision>
-        <xacro:inertial_cylinder mass="0.1" length="0.01" radius="0.045">
-            <origin xyz="0 0 0" rpy="0 0 0"/>
-        </xacro:inertial_cylinder>
-    </link>
-    <gazebo reference="back_left_wheel_link">
+                <cylinder radius="0.045" length="0.01"/>
+            </geometry>
+        </collision>
+        <xacro:inertial_cylinder mass="0.1" length="0.01" radius="0.045">
+            <origin xyz="0 0 0" rpy="0 0 0"/>
+        </xacro:inertial_cylinder>
+    </link>
+    <gazebo reference="back_right_wheel_link">
         <material>Gazebo/Black</material>
     </gazebo>
-    <!-- Gazebo specific elements -->
-    <!-- <gazebo>
-        <plugin name="gazebo_ros_control" filename="libgazebo_ros_control.so"/>
-    </gazebo> -->
 </robot>

Commit message: Finally i can do it. But yes no model.

File: src/robot_description/description/gazebo_control.xacro (robot description, xacro)
@@ -26,12 +26,12 @@
                 <param name="min">-5</param>
                 <param name="max">5</param>
-              </command_interface>
-              <state_interface name="position">
+            </command_interface>
+            <state_interface name="position">
                 <param name="initial_value">0.0</param>
-              </state_interface>
-              <state_interface name="velocity">
+            </state_interface>
+            <state_interface name="velocity">
                 <param name="initial_value">0.0</param>
-              </state_interface>
-              <state_interface name="effort"/>
+            </state_interface>
+            <state_interface name="effort"/>
         </joint>
         <!-- front_right_wheel -->
@@ -40,12 +40,12 @@
                 <param name="min">-5</param>
                 <param name="max">5</param>
-              </command_interface>
-              <state_interface name="position">
+            </command_interface>
+            <state_interface name="position">
                 <param name="initial_value">0.0</param>
-              </state_interface>
-              <state_interface name="velocity">
+            </state_interface>
+            <state_interface name="velocity">
                 <param name="initial_value">0.0</param>
-              </state_interface>
-              <state_interface name="effort"/>
+            </state_interface>
+            <state_interface name="effort"/>
         </joint>
         <!-- back_left_wheel -->
@@ -54,12 +54,12 @@
                 <param name="min">-5</param>
                 <param name="max">5</param>
-              </command_interface>
-              <state_interface name="position">
+            </command_interface>
+            <state_interface name="position">
                 <param name="initial_value">0.0</param>
-              </state_interface>
-              <state_interface name="velocity">
+            </state_interface>
+            <state_interface name="velocity">
                 <param name="initial_value">0.0</param>
-              </state_interface>
-              <state_interface name="effort"/>
+            </state_interface>
+            <state_interface name="effort"/>
         </joint>
         <!-- back_right_wheel -->
@@ -68,12 +68,34 @@
                 <param name="min">-5</param>
                 <param name="max">5</param>
-              </command_interface>
-              <state_interface name="position">
+            </command_interface>
+            <state_interface name="position">
                 <param name="initial_value">0.0</param>
-              </state_interface>
-              <state_interface name="velocity">
+            </state_interface>
+            <state_interface name="velocity">
                 <param name="initial_value">0.0</param>
-              </state_interface>
-              <state_interface name="effort"/>
+            </state_interface>
+            <state_interface name="effort"/>
+        </joint>
+        <!-- front_left_steering_joint -->
+        <joint name="front_left_steering_joint">
+            <command_interface name="position"/>
+            <state_interface name="position">
+                <param name="initial_value">0.0</param>
+            </state_interface>
+            <state_interface name="velocity">
+                <param name="initial_value">0.0</param>
+            </state_interface>
+            <state_interface name="effort"/>
+        </joint>
+        <!-- front_right_steering_joint -->
+        <joint name="front_right_steering_joint">
+            <command_interface name="position"/>
+            <state_interface name="position">
+                <param name="initial_value">0.0</param>
+            </state_interface>
+            <state_interface name="velocity">
+                <param name="initial_value">0.0</param>
+            </state_interface>
+            <state_interface name="effort"/>
         </joint>
     </ros2_control>

File: src/robot_description/description/robot_core.urdf.xacro (robot description, xacro)
@@ -1,3 +1,2 @@
-<?xml version="1.0"?>
 <robot xmlns:xacro="http://www.ros.org/wiki/xacro">
     <!-- Import the inertial macros -->
@@ -50,5 +49,5 @@
         </inertial>
     </link>
-    <joint name="front_left_wheel_steering_hinge" type="revolute">
+    <joint name="front_left_steering_joint" type="revolute">
         <origin xyz="0.10 0.07 0.045" rpy="0.0 0.0 0.0"/>
         <parent link="base_link"/>
@@ -56,4 +55,5 @@
         <axis xyz="0.0 0.0 1.0"/>
         <limit lower="-0.7854" upper="0.7854" effort="0.0" velocity="0.0"/>
+        <!-- <hardwareInterface>PositionJointInterface</hardwareInterface> -->
     </joint>
     <link name="front_left_wheel_link">
@@ -97,5 +97,5 @@
         </inertial>
     </link>
-    <joint name="front_right_wheel_steering_hinge" type="revolute">
+    <joint name="front_right_steering_joint" type="revolute">
         <origin xyz="0.10 -0.07 0.045" rpy="0.0 0.0 0.0"/>
         <parent link="base_link"/>
@@ -103,4 +103,5 @@
         <axis xyz="0.0 0.0 1.0"/>
         <limit lower="-0.7854" upper="0.7854" effort="0.0" velocity="0.0"/>
+        <!-- <hardwareInterface>PositionJointInterface</hardwareInterface> -->
     </joint>
     <link name="front_right_wheel_link">

Commit message: Add world launch on New Gazebo

File: src/robot_description/description/gazebo_control.xacro (robot description, xacro)
@@ -2,6 +2,6 @@
 <robot xmlns:xacro="http://www.ros.org/wiki/xacro" name="otto">
     <gazebo>
-        <plugin filename="libgazebo_ros2_control.so" name="gazebo_ros2_control">
-            <parameters>$(find robot_sim)/config/robot_controllers.yaml</parameters>
+         <plugin filename="gz_ros2_control-system" name="gz_ros2_control::GazeboSimROS2ControlPlugin">
+            <parameters>$(find robot_description)/config/robot_controllers.yaml</parameters>
         </plugin>
     </gazebo>
@@ -13,5 +13,5 @@
             </ros>
             <body_name>base_link</body_name>
-            <frameName>odom</frameName>            <!-- เปลี่ยนจาก world เป็น odom -->
+            <frameName>odom</frameName>
             <updateRate>100.0</updateRate>
         </plugin>
@@ -108,40 +108,49 @@
     <!-- base_link -->
     <gazebo reference="base_link">
-        <minDepth>0.0002</minDepth>
-        <kp value="1000000.0"/>
-        <kd value="100.0"/>
-        <material>Gazebo/Green</material>
+        <mu1>10</mu1>
+        <mu2>10</mu2>
+        <kp>10000000.0</kp>
+        <kd>1.0</kd>
+        <minDepth>0.01</minDepth>
+        <fdir1>1 0 0</fdir1>
+        <maxContacts value="64"/>
+    </gazebo>
+    <!-- Chassis -->
+    <gazebo reference="chassis">
+        <mu1>10</mu1>
+        <mu2>10</mu2>
+        <kp>10000000.0</kp>
+        <kd>1.0</kd>
+        <minDepth>0.01</minDepth>
+        <fdir1>1 0 0</fdir1>
+        <maxContacts value="64"/>
     </gazebo>
     <!-- front_left_wheel -->
     <gazebo reference="front_left_wheel">
-        <mu1>10.0</mu1>
-        <mu2>10.0</mu2>
-        <minDepth>0.0002</minDepth>
-        <kp value="1000000.0"/>
-        <kd value="100.0"/>
+        <mu1>0.5</mu1>
+        <mu2>0.5</mu2>
+        <kp>1000.0</kp>
+        <kd>1000.0</kd>
     </gazebo>
     <!-- front_right_wheel -->
     <gazebo reference="front_right_wheel">
-        <mu1>10.0</mu1>
-        <mu2>10.0</mu2>
-        <minDepth>0.0002</minDepth>
-        <kp value="1000000.0"/>
-        <kd value="100.0"/>
+        <mu1>0.5</mu1>
+        <mu2>0.5</mu2>
+        <kp>1000.0</kp>
+        <kd>1000.0</kd>
     </gazebo>
     <!-- back_left_wheel -->
     <gazebo reference="back_left_wheel">
-        <mu1>10.0</mu1>
-        <mu2>10.0</mu2>
-        <minDepth>0.0002</minDepth>
-        <kp value="1000000.0"/>
-        <kd value="100.0"/>
+        <mu1>0.5</mu1>
+        <mu2>0.5</mu2>
+        <kp>1000.0</kp>
+        <kd>1000.0</kd>
     </gazebo>
     <!-- back_right_wheel -->
     <gazebo reference="back_right_wheel">
-        <mu1>10.0</mu1>
-        <mu2>10.0</mu2>
-        <minDepth>0.0002</minDepth>
-        <kp value="1000000.0"/>
-        <kd value="100.0"/>
+        <mu1>0.5</mu1>
+        <mu2>0.5</mu2>
+        <kp>1000.0</kp>
+        <kd>1000.0</kd>
     </gazebo>
 </robot>
