Commit message: Again it' fail i can't run controller

File: src/robot_description/description/gazebo_control.xacro (robot description, xacro)
@@ -1,10 +1,5 @@
 <?xml version="1.0"?>
 <robot xmlns:xacro="http://www.ros.org/wiki/xacro" name="otto">
-    <gazebo>
-         <plugin filename="gz_ros2_control-system" name="gz_ros2_control::GazeboSimROS2ControlPlugin">
-            <parameters>$(find robot_description)/config/robot_controllers.yaml</parameters>
-        </plugin>
-    </gazebo>
-    <gazebo>
+     <!-- <gazebo>
         <plugin name="ground_truth_plugin" filename="libgazebo_ros_p3d.so">
             <ros>
@@ -12,7 +7,14 @@
                 <remapping>odom:=pose</remapping>
             </ros>
-            <body_name>base_link</body_name>
-            <frameName>odom</frameName>
+            <body_name>base_footprint</body_name>
+            <frameName>world</frameName>
             <updateRate>100.0</updateRate>
+        </plugin>
+    </gazebo> -->
+    <!-- ROS2 Control -->
+    <gazebo>
+    <!-- <plugin filename="libgazebo_ros2_control.so" name="gazebo_ros2_control"> -->
+        <plugin filename="gz_ros2_control-system" name="gz_ros2_control::GazeboSimROS2ControlPlugin">
+            <parameters>$(find robot_description)/config/robot_controllers.yaml</parameters>
         </plugin>
     </gazebo>
@@ -21,61 +23,5 @@
             <plugin>gazebo_ros2_control/GazeboSystem</plugin>
         </hardware>
-        <!-- front_left_wheel -->
-        <joint name="front_left_wheel">
-            <command_interface name="velocity">
-                <param name="min">-5</param>
-                <param name="max">5</param>
-            </command_interface>
-            <state_interface name="position">
-                <param name="initial_value">0.0</param>
-            </state_interface>
-            <state_interface name="velocity">
-                <param name="initial_value">0.0</param>
-            </state_interface>
-            <state_interface name="effort"/>
-        </joint>
-        <!-- front_right_wheel -->
-        <joint name="front_right_wheel">
-            <command_interface name="velocity">
-                <param name="min">-5</param>
-                <param name="max">5</param>
-            </command_interface>
-            <state_interface name="position">
-                <param name="initial_value">0.0</param>
-            </state_interface>
-            <state_interface name="velocity">
-                <param name="initial_value">0.0</param>
-            </state_interface>
-            <state_interface name="effort"/>
-        </joint>
-        <!-- back_left_wheel -->
-        <joint name="back_left_wheel">
-            <command_interface name="velocity">
-                <param name="min">-5</param>
-                <param name="max">5</param>
-            </command_interface>
-            <state_interface name="position">
-                <param name="initial_value">0.0</param>
-            </state_interface>
-            <state_interface name="velocity">
-                <param name="initial_value">0.0</param>
-            </state_interface>
-            <state_interface name="effort"/>
-        </joint>
-        <!-- back_right_wheel -->
-        <joint name="back_right_wheel">
-            <command_interface name="velocity">
-                <param name="min">-5</param>
-                <param name="max">5</param>
-            </command_interface>
-            <state_interface name="position">
-                <param name="initial_value">0.0</param>
-            </state_interface>
-            <state_interface name="velocity">
-                <param name="initial_value">0.0</param>
-            </state_interface>
-            <state_interface name="effort"/>
-        </joint>
-        <!-- front_left_steering_joint -->
+        <!-- Front Left Steering -->
         <joint name="front_left_steering_joint">
             <command_interface name="position">
@@ -91,5 +37,5 @@
             <state_interface name="effort"/>
         </joint>
-        <!-- front_right_steering_joint -->
+        <!-- Front Right Steering -->
         <joint name="front_right_steering_joint">
             <command_interface name="position">
@@ -105,7 +51,63 @@
             <state_interface name="effort"/>
         </joint>
+        <!-- Front Left Wheel -->
+        <joint name="front_left_wheel_joint">
+            <command_interface name="velocity">
+                <param name="min">-5</param>
+                <param name="max">5</param>
+            </command_interface>
+            <state_interface name="position">
+                <param name="initial_value">0.0</param>
+            </state_interface>
+            <state_interface name="velocity">
+                <param name="initial_value">0.0</param>
+            </state_interface>
+            <state_interface name="effort"/>
+        </joint>
+        <!-- Front Right Wheel -->
+        <joint name="front_right_wheel_joint">
+            <command_interface name="velocity">
+                <param name="min">-5</param>
+                <param name="max">5</param>
+            </command_interface>
+            <state_interface name="position">
+                <param name="initial_value">0.0</param>
+            </state_interface>
+            <state_interface name="velocity">
+                <param name="initial_value">0.0</param>
+            </state_interface>
+            <state_interface name="effort"/>
+        </joint>
+        <!-- Back Left Wheel -->
+        <joint name="back_left_wheel_joint">
+            <command_interface name="velocity">
+                <param name="min">-5</param>
+                <param name="max">5</param>
+            </command_interface>
+            <state_interface name="position">
+                <param name="initial_value">0.0</param>
+            </state_interface>
+            <state_interface name="velocity">
+                <param name="initial_value">0.0</param>
+            </state_interface>
+            <state_interface name="effort"/>
+        </joint>
+        <!-- Back Right Wheel -->
+        <joint name="back_right_wheel_joint">
+            <command_interface name="velocity">
+                <param name="min">-5</param>
+                <param name="max">5</param>
+            </command_interface>
+            <state_interface name="position">
+                <param name="initial_value">0.0</param>
+            </state_interface>
+            <state_interface name="velocity">
+                <param name="initial_value">0.0</param>
+            </state_interface>
+            <state_interface name="effort"/>
+        </joint>
     </ros2_control>
-    <!-- base_link -->
-    <gazebo reference="base_link">
+    <!-- Base Footprint Link -->
+    <gazebo reference="base_footprint">
         <mu1>10</mu1>
         <mu2>10</mu2>
@@ -117,5 +119,5 @@
     </gazebo>
     <!-- Chassis -->
-    <gazebo reference="chassis">
+    <gazebo reference="chassis_link">
         <mu1>10</mu1>
         <mu2>10</mu2>
@@ -126,6 +128,6 @@
         <maxContacts value="64"/>
     </gazebo>
-    <!-- front_left_wheel -->
-    <gazebo reference="front_left_wheel">
+    <!-- Front Left Wheel -->
+    <gazebo reference="front_left_wheel_link">
         <mu1>0.5</mu1>
         <mu2>0.5</mu2>
@@ -133,6 +135,6 @@
         <kd>1000.0</kd>
     </gazebo>
-    <!-- front_right_wheel -->
-    <gazebo reference="front_right_wheel">
+    <!-- Front Right Wheel -->
+    <gazebo reference="front_right_wheel_link">
         <mu1>0.5</mu1>
         <mu2>0.5</mu2>
@@ -140,6 +142,6 @@
         <kd>1000.0</kd>
     </gazebo>
-    <!-- back_left_wheel -->
-    <gazebo reference="back_left_wheel">
+    <!-- Back Left Wheel -->
+    <gazebo reference="back_left_wheel_link">
         <mu1>0.5</mu1>
         <mu2>0.5</mu2>
@@ -147,6 +149,6 @@
         <kd>1000.0</kd>
     </gazebo>
-    <!-- back_right_wheel -->
-    <gazebo reference="back_right_wheel">
+    <!-- Back Right Wheel -->
+    <gazebo reference="back_right_wheel_link">
         <mu1>0.5</mu1>
         <mu2>0.5</mu2>

File: src/robot_description/description/limo_core.urdf.xacro (robot description, xacro)
@@ -1,187 +1,174 @@
-<robot xmlns:xacro="http://www.ros.org/wiki/xacro">
-    <!-- Import the inertial macros -->
+<?xml version="1.0"?>
+<robot name="limo" xmlns:xacro="http://ros.org/wiki/xacro">
+    <!-- Import macros -->
     <xacro:include filename="inertial_macros.xacro"/>
-    <!-- COLOR NAME  -->
-    <material name="white">
-        <color rgba="1 1 1 1" />
-    </material>
-    <material name="black">
-        <color rgba="0 0 0 1"/>
-    </material>
-    <material name="blue">
-        <color rgba="0 0 1 1"/>
-    </material>
-    <material name="red">
-        <color rgba="1 0 0 1"/>
-    </material>
-    <!-- base link -->
-    <link name="base_link"/>
-    <!-- chassis link -->
-    <joint name="chassis_joint" type="fixed">
-        <origin xyz="-0.1 0.0 0.0" rpy="0.0 0.0 0.0"/>
-        <parent link="base_link"/>
-        <child link="chassis"/>
-    </joint>
-    <link name="chassis">
-        <visual name="">
-            <origin xyz="0.1 0.0 -0.05" rpy="0.0 0.0 1.57"/>
-            <geometry>
-                <mesh filename="file://$(find ${description_package})/meshes/limo_base.dae"/>
-            </geometry>
-            <!-- <material name="white"/> -->
-        </visual>
-        <collision>
-            <origin xyz="0.075 0.0 0.045" rpy="0.0 0.0 0.0"/>
-            <geometry>
-                <box size="0.15 0.13 0.1"/>
-            </geometry>
-        </collision>
-        <xacro:inertial_box mass="5.5" x="0.2" y="0.13" z="0.1">
-             <origin xyz="0.1 0 0.045" rpy="0 0 0"/>
-        </xacro:inertial_box>
-    </link>
-    <!-- <gazebo reference="chassis">
-        <material>Gazebo/White</material>
-    </gazebo> -->
-    <!-- front left wheel -->
-    <link name="front_left_wheel_joint_link">
-        <inertial>
-            <origin xyz="0.0 0.0 0.0" rpy="0.0 0.0 0.0"/>
-            <mass value="0.1"/>
-            <inertia ixx="0.01" ixy="0.0" ixz="0.0" iyy="0.01" iyz="0.0" izz="0.01"/>
-        </inertial>
-    </link>
-    <joint name="front_left_steering_joint" type="revolute">
-        <origin xyz="0.1 0.07 0.0" rpy="0.0 0.0 0.0"/>
-        <parent link="base_link"/>
-        <child link="front_left_wheel_joint_link"/>
-        <axis xyz="0.0 0.0 1.0"/>
-        <limit lower="-0.7854" upper="0.7854" effort="10.0" velocity="3.0"/>
-    </joint>
-    <link name="front_left_wheel_link">
-        <visual name="">
-            <origin xyz="0.0 0.0 -0.005" rpy="1.57 0.0 0.0"/>
-            <geometry>
-                <mesh filename="file://$(find ${description_package})/meshes/limo_wheel.dae"/>
-            </geometry>
-            <!-- <material name="blue"/> -->
-        </visual>
-        <collision>
-            <!-- <origin xyz="0.0 0.0 0.0" rpy="0.0 0.0 0.0"/> -->
-            <geometry>
-                <cylinder radius="0.045" length="0.01"/>
-            </geometry>
-        </collision>
-        <xacro:inertial_cylinder mass="0.1" length="0.01" radius="0.045">
+    <!-- Base Footprint Link -->
+        <link name="base_footprint"/>
+    <!-- Chassis -->
+        <!-- Joint -->
+        <joint name="chassis_joint" type="fixed">
+            <origin xyz="0 0 0.15" rpy="0 0 0"/>
+            <parent link="base_footprint"/>
+            <child link="chassis_link"/>
+        </joint>
+        <!-- Link -->
+        <link name="chassis_link">
+            <visual name="">
+                <origin xyz="0 0 -0.15" rpy="0 0 1.57" />
+                <geometry>
+                    <mesh filename="file://$(find robot_description)/meshes/limo_optimal.dae" scale="1 1 1"/>
+                </geometry>
+            </visual>
+            <collision>
+                <origin xyz="0 0 0" rpy="0 0 0"/>
+                <geometry>
+                    <box size="0.20 0.13 0.1"/>
+                </geometry>
+            </collision>
+            <xacro:inertial_box mass="2.0" x="0.2" y="0.13" z="0.1">
+                <origin xyz="0 0 0" rpy="0 0 0"/>
+            </xacro:inertial_box>
+        </link>
+    <!-- Front Left Steering -->
+        <!-- Link -->
+        <link name="front_left_steering_link">
+            <inertial>
+                <origin xyz="0 0 0" rpy="0 0 0"/>
+                <mass value="0.1"/>
+                <inertia ixx="0.01" ixy="0.0" ixz="0.0" iyy="0.01" iyz="0.0" izz="0.01"/>
+            </inertial>
+        </link>
+        <!-- Joint -->
+        <joint name="front_left_steering_joint" type="revolute">
+            <origin xyz="0.1 0.07 -0.1" rpy="0 0 0"/>
+            <parent link="chassis_link"/>
+            <child link="front_left_steering_link"/>
+            <axis xyz="0 0 1"/>
+            <limit lower="-0.523598767" upper="0.523598767" effort="1000" velocity="1.0" />
+        </joint>
+    <!-- Front Left Wheel -->
+        <!-- Link -->
+        <link name="front_left_wheel_link">
+            <visual>
+              <origin xyz="0 0 0" rpy="0 0 0"/>
+              <geometry>
+                  <mesh filename="file://$(find robot_description)/meshes/limo_optimal_wheels.dae" scale="1 1 1"/>
+              </geometry>
+            </visual>
+            <collision>
+                <origin xyz="0 0.005 0" rpy="1.57 0 0"/>
+                <geometry>
+                    <cylinder radius="0.045" length="0.01"/>
+                </geometry>
+            </collision>
+            <xacro:inertial_cylinder mass="0.25" length="0.01" radius="0.045">
+                <origin xyz="0 0 0" rpy="0 0 0"/>
+            </xacro:inertial_cylinder>
+        </link>
+        <!-- Joint -->
+        <joint name="front_left_wheel_joint" type="continuous">
             <origin xyz="0 0 0" rpy="0 0 0"/>
-        </xacro:inertial_cylinder>
-    </link>
-    <joint name="front_left_wheel" type="continuous">
-        <origin xyz="0.0 0.0 0.0" rpy="-1.57 0.0 0.0"/>
-        <parent link="front_left_wheel_joint_link"/>
-        <child link="front_left_wheel_link"/>
-        <axis xyz="0.0 0.0 1.0"/>
-    </joint>
-    <!-- <gazebo reference="front_left_wheel_link">
-        <material>Gazebo/Blue</material>
-    </gazebo> -->
-    <!-- front right wheel -->
-    <link name="front_right_wheel_joint_link">
-        <inertial>
-            <origin xyz="0.0 0.0 0.0" rpy="0.0 0.0 0.0"/>
-            <mass value="0.1"/>
-            <inertia ixx="0.01" ixy="0.0" ixz="0.0" iyy="0.01" iyz="0.0" izz="0.01"/>
-        </inertial>
-    </link>
-    <joint name="front_right_steering_joint" type="revolute">
-        <origin xyz="0.1 -0.07 0.0" rpy="0.0 0.0 0.0"/>
-        <parent link="base_link"/>
-        <child link="front_right_wheel_joint_link"/>
-        <axis xyz="0.0 0.0 1.0"/>
-        <limit lower="-0.785" upper="0.785" effort="10.0" velocity="3.0"/>
-    </joint>
-    <link name="front_right_wheel_link">
-        <visual name="">
-            <origin xyz="0.0 0.0 -0.005" rpy="1.57 0.0 0.0"/>
-            <geometry>
-                <mesh filename="file://$(find ${description_package})/meshes/limo_wheel.dae"/>
-            </geometry>
-            <!-- <material name="blue"/> -->
-        </visual>
-        <collision>
-            <!-- <origin xyz="0.0 0.0 0.0" rpy="0.0 0.0 0.0"/> -->
-            <geometry>
-                <cylinder radius="0.045" length="0.01"/>
-            </geometry>
-        </collision>
-        <xacro:inertial_cylinder mass="0.1" length="0.01" radius="0.045">
+            <parent link="front_left_steering_link"/>
+            <child link="front_left_wheel_link"/>
+            <axis xyz="0 1 0"/>
+            <limit effort="100.0" velocity="10.0"/>
+        </joint>
+    <!-- Front Right Steering -->
+        <!-- Link -->
+        <link name="front_right_steering_link">
+            <inertial>
+                <origin xyz="0 0 0" rpy="0 0 0"/>
+                <mass value="0.1"/>
+                <inertia ixx="0.01" ixy="0.0" ixz="0.0" iyy="0.01" iyz="0.0" izz="0.01"/>
+            </inertial>
+        </link>
+        <!-- Joint -->
+        <joint name="front_right_steering_joint" type="revolute">
+            <origin xyz="0.1 -0.07 -0.1" rpy="3.14159 0 0"/>
+            <parent link="chassis_link"/>
+            <child link="front_right_steering_link"/>
+            <axis xyz="0 0 -1"/>
+            <limit lower="-0.523598767" upper="0.523598767" effort="1000" velocity="1.0" />
+        </joint>
+    <!-- Front Right Wheel -->
+        <!-- Link -->
+        <link name="front_right_wheel_link">
+            <visual>
+              <origin xyz="0 0 0" rpy="0 0 0" />
+              <geometry>
+                  <mesh filename="file://$(find robot_description)/meshes/limo_optimal_wheels.dae" scale="1 1 1"/>
+              </geometry>
+            </visual>
+            <collision>
+                <origin xyz="0 0.005 0" rpy="1.57 0 0"/>
+                <geometry>
+                    <cylinder radius="0.045" length="0.01"/>
+                </geometry>
+            </collision>
+            <xacro:inertial_cylinder mass="0.25" length="0.01" radius="0.045">
+                <origin xyz="0 0 0" rpy="0 0 0"/>
+            </xacro:inertial_cylinder>
+        </link>
+        <!-- Joint -->
+        <joint name="front_right_wheel_joint" type="continuous">
             <origin xyz="0 0 0" rpy="0 0 0"/>
-        </xacro:inertial_cylinder>
-    </link>
-    <joint name="front_right_wheel" type="continuous">
-        <origin xyz="0.0 0.0 0.0" rpy="1.57 0.0 0.0"/>
-        <parent link="front_right_wheel_joint_link"/>
-        <child link="front_right_wheel_link"/>
-        <axis xyz="0.0 0.0 -1.0"/>
-    </joint>
-    <!-- <gazebo reference="front_right_wheel_link">
-        <material>Gazebo/Blue</material>
-    </gazebo> -->
-    <!-- back left wheel -->
-    <joint name="back_left_wheel" type="continuous">
-        <origin xyz="-0.1 0.07 0.0" rpy="-1.57 0.0 0.0"/>
-        <parent link="base_link"/>
-        <child link="back_left_wheel_link"/>
-        <axis xyz="0.0 0.0 1.0"/>
-    </joint>
-    <link name="back_left_wheel_link">
-        <visual name="">
-            <origin xyz="0 0 -0.005" rpy="1.57 0 0"/>
-            <geometry>
-                <mesh filename="file://$(find ${description_package})/meshes/limo_wheel.dae"/>
-            </geometry>
-            <!-- <material name="black"/> -->
-        </visual>
-        <collision>
-            <!-- <origin xyz="0.0 0.0 0.0" rpy="0.0 0.0 0.0"/> -->
-            <geometry>
-                <cylinder radius="0.045" length="0.01"/>
-            </geometry>
-        </collision>
-        <xacro:inertial_cylinder mass="0.1" length="0.01" radius="0.045">
-            <origin xyz="0 0 0" rpy="0 0 0"/>
-        </xacro:inertial_cylinder>
-    </link>
-    <!-- <gazebo reference="back_left_wheel_link">
-        <material>Gazebo/Black</material>
-    </gazebo> -->
-    <!-- back right wheel -->
-    <joint name="back_right_wheel" type="continuous">
-        <origin xyz="-0.1 -0.07 0" rpy="1.57 0 0" />
-        <parent link="base_link"/>
-        <child link="back_right_wheel_link"/>
-        <axis xyz="0.0 0.0 -1.0"/>
-        <limit lower="0.0" upper="0.0" effort="0.0" velocity="0.0"/>
-    </joint>
-    <link name="back_right_wheel_link">
-        <visual name="">
-            <origin xyz="0 0 -0.005" rpy="1.57 0 0"/>
-            <geometry>
-                <mesh filename="file://$(find ${description_package})/meshes/limo_wheel.dae"/>
-            </geometry>
-            <!-- <material name="black"/> -->
-        </visual>
-        <collision>
-            <!-- <origin xyz="0.0 0.0 0.0" rpy="0.0 0.0 0.0"/> -->
-            <geometry>
-                <cylinder radius="0.045" length="0.01"/>
-            </geometry>
-        </collision>
-        <xacro:inertial_cylinder mass="0.1" length="0.01" radius="0.045">
-            <origin xyz="0 0 0" rpy="0 0 0"/>
-        </xacro:inertial_cylinder>
-    </link>
-    <!-- <gazebo reference="back_right_wheel_link">
-        <material>Gazebo/Black</material>
-    </gazebo> -->
+            <parent link="front_right_steering_link"/>
+            <child link="front_right_wheel_link"/>
+            <axis xyz="0 -1 0"/>
+            <limit effort="100.0" velocity="10.0"/>
+        </joint>
+    <!-- Back Left Wheel -->
+        <!-- Link -->
+        <link name="back_left_wheel_link">
+            <visual>
+              <origin xyz="0 0 0" rpy="0 0 0"/>
+              <geometry>
+                  <mesh filename="file://$(find robot_description)/meshes/limo_optimal_wheels.dae" scale="1 1 1"/>
+              </geometry>
+            </visual>
+            <collision>
+                <origin xyz="0 0.005 0" rpy="1.57 0 0"/>
+                <geometry>
+                    <cylinder radius="0.045" length="0.01"/>
+                </geometry>
+            </collision>
+            <xacro:inertial_cylinder mass="0.25" length="0.01" radius="0.045">
+                <origin xyz="0 0 0" rpy="0 0 0"/>
+            </xacro:inertial_cylinder>
+        </link>
+        <!-- Joint -->
+        <joint name="back_left_wheel_joint" type="continuous">
+            <origin xyz="-0.1 0.07 -0.1" rpy="0 0.0 0.0"/>
+            <parent link="chassis_link"/>
+            <child link="back_left_wheel_link"/>
+            <axis xyz="0 1 0"/>
+            <limit effort="100.0" velocity="10.0"/>
+        </joint>
+    <!-- Back Right Wheel -->
+        <!-- Link -->
+        <link name="back_right_wheel_link">
+            <visual>
+              <origin xyz="0 0 0" rpy="0 0 0"/>
+              <geometry>
+                  <mesh filename="file://$(find robot_description)/meshes/limo_optimal_wheels.dae" scale="1 1 1"/>
+              </geometry>
+            </visual>
+            <collision>
+                <origin xyz="0 0.005 0" rpy="1.57 0 0"/>
+                <geometry>
+                    <cylinder radius="0.045" length="0.01"/>
+                </geometry>
+            </collision>
+            <xacro:inertial_cylinder mass="0.25" length="0.01" radius="0.045">
+                <origin xyz="0 0 0" rpy="0 0 0"/>
+            </xacro:inertial_cylinder>
+        </link>
+        <!-- Joint -->
+        <joint name="back_right_wheel_joint" type="continuous">
+            <origin xyz="-0.1 -0.07 -0.1" rpy="3.14159 0 0"/>
+            <parent link="chassis_link"/>
+            <child link="back_right_wheel_link"/>
+            <axis xyz="0 -1 0"/>
+            <limit effort="100.0" velocity="10.0"/>
+        </joint>
 </robot>
