Commit message: Again it' fail i can't run controller

File: src/robot_description/description/robot-main.xacro (robot description, xacro)
@@ -2,9 +2,5 @@
 <robot xmlns:xacro="http://www.ros.org/wiki/xacro"  name="fake-limo">
     <xacro:property name="description_package" value="robot_description"/>
-    <!-- <xacro:include filename="$(find robot_description)/description/robot_core.urdf.xacro"/> -->
     <xacro:include filename="$(find robot_description)/description/limo_core.urdf.xacro"/>
     <xacro:include filename="$(find robot_description)/description/gazebo_control.xacro"/>
-    <!-- <xacro:include filename="$(find robot_description)/description/camera.xacro"/> -->
-    <!-- <xacro:include filename="$(find robot_description)/description/lidar.xacro"/> -->
-    <!-- <xacro:include filename="$(find robot_description)/description/imu.xacro"/> -->
 </robot>
