Commit message: Add limo_models to my project

File: src/robot_description/description/limo_core.urdf.xacro (robot description, xacro)
@@ -19,5 +19,5 @@
     <!-- chassis link -->
     <joint name="chassis_joint" type="fixed">
-        <origin xyz="0.0 0.0 0.095" rpy="0.0 0.0 0.0"/>
+        <origin xyz="-0.1 0.0 0.0" rpy="0.0 0.0 0.0"/>
         <parent link="base_link"/>
         <child link="chassis"/>
@@ -25,18 +25,18 @@
     <link name="chassis">
         <visual name="">
-            <origin xyz="0.0 0.0 0.0" rpy="0.0 0.0 0.0"/>
+            <origin xyz="0.1 0.0 -0.05" rpy="0.0 0.0 1.57"/>
             <geometry>
-                <box size="0.20 0.13 0.1"/>
+                <mesh filename="file://$(find ${description_package})/meshes/limo_base.dae"/>
             </geometry>
             <material name="white"/>
         </visual>
         <collision>
-            <origin xyz="0.0 0.0 0.0" rpy="0.0 0.0 0.0"/>
+            <origin xyz="0.075 0.0 0.045" rpy="0.0 0.0 0.0"/>
             <geometry>
-                <box size="0.20 0.13 0.1"/>
+                <box size="0.15 0.13 0.1"/>
             </geometry>
         </collision>
-        <xacro:inertial_box mass="3.0" x="0.13" y="0.2" z="0.1">
-            <origin xyz="0.0 0.0 0.0" rpy="0 0 0"/>
+        <xacro:inertial_box mass="5.5" x="0.2" y="0.13" z="0.1">
+             <origin xyz="0.1 0 0.045" rpy="0 0 0"/>
         </xacro:inertial_box>
     </link>
@@ -53,20 +53,20 @@
     </link>
     <joint name="front_left_steering_joint" type="revolute">
-        <origin xyz="0.10 0.07 -0.045" rpy="0.0 0.0 0.0"/>
-        <parent link="chassis"/>
+        <origin xyz="0.1 0.07 0.0" rpy="0.0 0.0 0.0"/>
+        <parent link="base_link"/>
         <child link="front_left_wheel_joint_link"/>
         <axis xyz="0.0 0.0 1.0"/>
-        <limit lower="-0.7854" upper="0.7854" effort="0.0" velocity="0.0"/>
+        <limit lower="-0.7854" upper="0.7854" effort="10.0" velocity="3.0"/>
     </joint>
     <link name="front_left_wheel_link">
         <visual name="">
-            <origin xyz="0.0 0.0 0.0" rpy="0.0 0.0 0.0"/>
+            <origin xyz="0.0 0.0 -0.005" rpy="1.57 0.0 0.0"/>
             <geometry>
-                <cylinder radius="0.045" length="0.01"/>
+                <mesh filename="file://$(find ${description_package})/meshes/limo_wheel.dae"/>
             </geometry>
             <material name="blue"/>
         </visual>
         <collision>
-            <origin xyz="0.0 0.0 0.0" rpy="0.0 0.0 0.0"/>
+            <!-- <origin xyz="0.0 0.0 0.0" rpy="0.0 0.0 0.0"/> -->
             <geometry>
                 <cylinder radius="0.045" length="0.01"/>
@@ -95,20 +95,20 @@
     </link>
     <joint name="front_right_steering_joint" type="revolute">
-        <origin xyz="0.10 -0.07 -0.045" rpy="0.0 0.0 0.0"/>
-        <parent link="chassis"/>
+        <origin xyz="0.1 -0.07 0.0" rpy="0.0 0.0 0.0"/>
+        <parent link="base_link"/>
         <child link="front_right_wheel_joint_link"/>
         <axis xyz="0.0 0.0 1.0"/>
-        <limit lower="-0.7854" upper="0.7854" effort="0.0" velocity="0.0"/>
+        <limit lower="-0.785" upper="0.785" effort="10.0" velocity="3.0"/>
     </joint>
     <link name="front_right_wheel_link">
         <visual name="">
-            <origin xyz="0.0 0.0 0.0" rpy="0.0 0.0 0.0"/>
+            <origin xyz="0.0 0.0 -0.005" rpy="1.57 0.0 0.0"/>
             <geometry>
-                <cylinder radius="0.045" length="0.01"/>
+                <mesh filename="file://$(find ${description_package})/meshes/limo_wheel.dae"/>
             </geometry>
             <material name="blue"/>
         </visual>
         <collision>
-            <origin xyz="0.0 0.0 0.0" rpy="0.0 0.0 0.0"/>
+            <!-- <origin xyz="0.0 0.0 0.0" rpy="0.0 0.0 0.0"/> -->
             <geometry>
                 <cylinder radius="0.045" length="0.01"/>
@@ -120,8 +120,8 @@
     </link>
     <joint name="front_right_wheel" type="continuous">
-        <origin xyz="0.0 0.0 0.0" rpy="-1.57 0.0 0.0"/>
+        <origin xyz="0.0 0.0 0.0" rpy="1.57 0.0 0.0"/>
         <parent link="front_right_wheel_joint_link"/>
         <child link="front_right_wheel_link"/>
-        <axis xyz="0.0 0.0 1.0"/>
+        <axis xyz="0.0 0.0 -1.0"/>
     </joint>
     <gazebo reference="front_right_wheel_link">
@@ -130,6 +130,6 @@
     <!-- back left wheel -->
     <joint name="back_left_wheel" type="continuous">
-        <origin xyz="-0.10 0.07 -0.045" rpy="-1.57 0.0 0.0"/>
-        <parent link="chassis"/>
+        <origin xyz="-0.1 0.07 0.0" rpy="-1.57 0.0 0.0"/>
+        <parent link="base_link"/>
         <child link="back_left_wheel_link"/>
         <axis xyz="0.0 0.0 1.0"/>
@@ -137,12 +137,12 @@
     <link name="back_left_wheel_link">
         <visual name="">
-            <origin xyz="0.0 0.0 0.0" rpy="0.0 0.0 0.0"/>
+            <origin xyz="0 0 -0.005" rpy="1.57 0 0"/>
             <geometry>
-                <cylinder radius="0.045" length="0.01"/>
+                <mesh filename="file://$(find ${description_package})/meshes/limo_wheel.dae"/>
             </geometry>
             <material name="black"/>
         </visual>
         <collision>
-            <origin xyz="0.0 0.0 0.0" rpy="0.0 0.0 0.0"/>
+            <!-- <origin xyz="0.0 0.0 0.0" rpy="0.0 0.0 0.0"/> -->
             <geometry>
                 <cylinder radius="0.045" length="0.01"/>
@@ -158,20 +158,20 @@
     <!-- back right wheel -->
     <joint name="back_right_wheel" type="continuous">
-        <origin xyz="-0.10 -0.07 -0.045" rpy="-1.57 0.0 0.0"/>
-        <parent link="chassis"/>
+        <origin xyz="-0.1 -0.07 0" rpy="1.57 0 0" />
+        <parent link="base_link"/>
         <child link="back_right_wheel_link"/>
-        <axis xyz="0.0 0.0 1.0"/>
+        <axis xyz="0.0 0.0 -1.0"/>
         <limit lower="0.0" upper="0.0" effort="0.0" velocity="0.0"/>
     </joint>
     <link name="back_right_wheel_link">
         <visual name="">
-            <origin xyz="0.0 0.0 0.0" rpy="0.0 0.0 0.0"/>
+            <origin xyz="0 0 -0.005" rpy="1.57 0 0"/>
             <geometry>
-                <cylinder radius="0.045" length="0.01"/>
+                <mesh filename="file://$(find ${description_package})/meshes/limo_wheel.dae"/>
             </geometry>
             <material name="black"/>
         </visual>
         <collision>
-            <origin xyz="0.0 0.0 0.0" rpy="0.0 0.0 0.0"/>
+            <!-- <origin xyz="0.0 0.0 0.0" rpy="0.0 0.0 0.0"/> -->
             <geometry>
                 <cylinder radius="0.045" length="0.01"/>

File: src/robot_description/description/robot-main.xacro (robot description, xacro)
@@ -1,8 +1,10 @@
 <?xml version="1.0"?>
 <robot xmlns:xacro="http://www.ros.org/wiki/xacro"  name="fake-limo">
-    <xacro:include filename="robot_core.urdf.xacro"/>
-    <xacro:include filename="gazebo_control.xacro"/>
-    <xacro:include filename="camera.xacro"/>
-    <xacro:include filename="lidar.xacro"/>
-    <xacro:include filename="imu.xacro"/>
+    <xacro:property name="description_package" value="robot_description"/>
+    <!-- <xacro:include filename="$(find robot_description)/description/robot_core.urdf.xacro"/> -->
+    <xacro:include filename="$(find robot_description)/description/limo_core.urdf.xacro"/>
+    <xacro:include filename="$(find robot_description)/description/gazebo_control.xacro"/>
+    <!-- <xacro:include filename="$(find robot_description)/description/camera.xacro"/> -->
+    <!-- <xacro:include filename="$(find robot_description)/description/lidar.xacro"/> -->
+    <!-- <xacro:include filename="$(find robot_description)/description/imu.xacro"/> -->
 </robot>

Commit message: Update InvertKinematic

File: src/robot_description/description/limo_core.urdf.xacro (robot description, xacro)
@@ -29,5 +29,5 @@
                 <mesh filename="file://$(find ${description_package})/meshes/limo_base.dae"/>
             </geometry>
-            <material name="white"/>
+            <!-- <material name="white"/> -->
         </visual>
         <collision>
@@ -41,7 +41,7 @@
         </xacro:inertial_box>
     </link>
-    <gazebo reference="chassis">
+    <!-- <gazebo reference="chassis">
         <material>Gazebo/White</material>
-    </gazebo>
+    </gazebo> -->
     <!-- front left wheel -->
     <link name="front_left_wheel_joint_link">
@@ -65,5 +65,5 @@
                 <mesh filename="file://$(find ${description_package})/meshes/limo_wheel.dae"/>
             </geometry>
-            <material name="blue"/>
+            <!-- <material name="blue"/> -->
         </visual>
         <collision>
@@ -83,7 +83,7 @@
         <axis xyz="0.0 0.0 1.0"/>
     </joint>
-    <gazebo reference="front_left_wheel_link">
+    <!-- <gazebo reference="front_left_wheel_link">
         <material>Gazebo/Blue</material>
-    </gazebo>
+    </gazebo> -->
     <!-- front right wheel -->
     <link name="front_right_wheel_joint_link">
@@ -107,5 +107,5 @@
                 <mesh filename="file://$(find ${description_package})/meshes/limo_wheel.dae"/>
             </geometry>
-            <material name="blue"/>
+            <!-- <material name="blue"/> -->
         </visual>
         <collision>
@@ -125,7 +125,7 @@
         <axis xyz="0.0 0.0 -1.0"/>
     </joint>
-    <gazebo reference="front_right_wheel_link">
+    <!-- <gazebo reference="front_right_wheel_link">
         <material>Gazebo/Blue</material>
-    </gazebo>
+    </gazebo> -->
     <!-- back left wheel -->
     <joint name="back_left_wheel" type="continuous">
@@ -141,5 +141,5 @@
                 <mesh filename="file://$(find ${description_package})/meshes/limo_wheel.dae"/>
             </geometry>
-            <material name="black"/>
+            <!-- <material name="black"/> -->
         </visual>
         <collision>
@@ -153,7 +153,7 @@
         </xacro:inertial_cylinder>
     </link>
-    <gazebo reference="back_left_wheel_link">
+    <!-- <gazebo reference="back_left_wheel_link">
         <material>Gazebo/Black</material>
-    </gazebo>
+    </gazebo> -->
     <!-- back right wheel -->
     <joint name="back_right_wheel" type="continuous">
@@ -170,5 +170,5 @@
                 <mesh filename="file://$(find ${description_package})/meshes/limo_wheel.dae"/>
             </geometry>
-            <material name="black"/>
+            <!-- <material name="black"/> -->
         </visual>
         <collision>
@@ -182,6 +182,6 @@
         </xacro:inertial_cylinder>
     </link>
-    <gazebo reference="back_right_wheel_link">
+    <!-- <gazebo reference="back_right_wheel_link">
         <material>Gazebo/Black</material>
-    </gazebo>
+    </gazebo> -->
 </robot>

Commit message: Remove commented material references from limo_core.urdf.xacro

File: src/robot_description/description/limo_core.urdf.xacro (robot description, xacro)
@@ -16,5 +16,4 @@
                 <mesh filename="file://$(find ${description_package})/meshes/limo_optimal.dae"/>
             </geometry>
-            <!-- <material name="white"/> -->
         </visual>
         <collision>
@@ -28,7 +27,4 @@
         </xacro:inertial_box>
     </link>
-    <!-- <gazebo reference="chassis">
-        <material>Gazebo/White</material>
-    </gazebo> -->
     <!-- front left wheel -->
     <link name="front_left_wheel_joint_link">
