Commit message: Update Gazebo config

File: src/robot_description/description/camera.xacro (robot description, xacro)
@@ -4,5 +4,5 @@
         <parent link="chassis"/>
         <child link="camera_link"/>
-        <origin xyz="0.105 0.0 0.035" rpy="0 0 0"/>
+        <origin xyz="0.190 0.0 0.135" rpy="0 0 0"/>
     </joint>
     <link name="camera_link">

File: src/robot_description/description/gazebo_control.xacro (robot description, xacro)
@@ -108,40 +108,49 @@
     <!-- base_link -->
     <gazebo reference="base_link">
-        <minDepth>0.0002</minDepth>
-        <kp value="1000000.0"/>
-        <kd value="100.0"/>
-        <material>Gazebo/Green</material>
+        <mu1>10</mu1>
+        <mu2>10</mu2>
+        <kp>10000000.0</kp>
+        <kd>1.0</kd>
+        <minDepth>0.01</minDepth>
+        <fdir1>1 0 0</fdir1>
+        <maxContacts value="64"/>
+    </gazebo>
+    <!-- Chassis -->
+    <gazebo reference="chassis">
+        <mu1>10</mu1>
+        <mu2>10</mu2>
+        <kp>10000000.0</kp>
+        <kd>1.0</kd>
+        <minDepth>0.01</minDepth>
+        <fdir1>1 0 0</fdir1>
+        <maxContacts value="64"/>
     </gazebo>
     <!-- front_left_wheel -->
     <gazebo reference="front_left_wheel">
-        <mu1>10.0</mu1>
-        <mu2>10.0</mu2>
-        <minDepth>0.0002</minDepth>
-        <kp value="1000000.0"/>
-        <kd value="100.0"/>
+        <mu1>0.5</mu1>
+        <mu2>0.5</mu2>
+        <kp>1000.0</kp>
+        <kd>1000.0</kd>
     </gazebo>
     <!-- front_right_wheel -->
     <gazebo reference="front_right_wheel">
-        <mu1>10.0</mu1>
-        <mu2>10.0</mu2>
-        <minDepth>0.0002</minDepth>
-        <kp value="1000000.0"/>
-        <kd value="100.0"/>
+        <mu1>0.5</mu1>
+        <mu2>0.5</mu2>
+        <kp>1000.0</kp>
+        <kd>1000.0</kd>
     </gazebo>
     <!-- back_left_wheel -->
     <gazebo reference="back_left_wheel">
-        <mu1>10.0</mu1>
-        <mu2>10.0</mu2>
-        <minDepth>0.0002</minDepth>
-        <kp value="1000000.0"/>
-        <kd value="100.0"/>
+        <mu1>0.5</mu1>
+        <mu2>0.5</mu2>
+        <kp>1000.0</kp>
+        <kd>1000.0</kd>
     </gazebo>
     <!-- back_right_wheel -->
     <gazebo reference="back_right_wheel">
-        <mu1>10.0</mu1>
-        <mu2>10.0</mu2>
-        <minDepth>0.0002</minDepth>
-        <kp value="1000000.0"/>
-        <kd value="100.0"/>
+        <mu1>0.5</mu1>
+        <mu2>0.5</mu2>
+        <kp>1000.0</kp>
+        <kd>1000.0</kd>
     </gazebo>
 </robot>

File: src/robot_description/description/limo_core.urdf.xacro (robot description, xacro)
@@ -2,17 +2,4 @@
     <!-- Import the inertial macros -->
     <xacro:include filename="inertial_macros.xacro"/>
-    <!-- COLOR NAME  -->
-    <material name="white">
-        <color rgba="1 1 1 1" />
-    </material>
-    <material name="black">
-        <color rgba="0 0 0 1"/>
-    </material>
-    <material name="blue">
-        <color rgba="0 0 1 1"/>
-    </material>
-    <material name="red">
-        <color rgba="1 0 0 1"/>
-    </material>
     <!-- base link -->
     <link name="base_link"/>
@@ -27,5 +14,5 @@
             <origin xyz="0.1 0.0 -0.05" rpy="0.0 0.0 1.57"/>
             <geometry>
-                <mesh filename="file://$(find ${description_package})/meshes/limo_base.dae"/>
+                <mesh filename="file://$(find ${description_package})/meshes/limo_optimal.dae"/>
             </geometry>
             <!-- <material name="white"/> -->
@@ -37,6 +24,6 @@
             </geometry>
         </collision>
-        <xacro:inertial_box mass="5.5" x="0.2" y="0.13" z="0.1">
-             <origin xyz="0.1 0 0.045" rpy="0 0 0"/>
+        <xacro:inertial_box mass="2.0" x="0.2" y="0.13" z="0.1">
+            <origin xyz="0 0 0" rpy="0 0 0"/>
         </xacro:inertial_box>
     </link>
@@ -63,15 +50,13 @@
             <origin xyz="0.0 0.0 -0.005" rpy="1.57 0.0 0.0"/>
             <geometry>
-                <mesh filename="file://$(find ${description_package})/meshes/limo_wheel.dae"/>
+                <mesh filename="file://$(find ${description_package})/meshes/limo_optimal_wheels.dae"/>
             </geometry>
-            <!-- <material name="blue"/> -->
         </visual>
         <collision>
-            <!-- <origin xyz="0.0 0.0 0.0" rpy="0.0 0.0 0.0"/> -->
             <geometry>
                 <cylinder radius="0.045" length="0.01"/>
             </geometry>
         </collision>
-        <xacro:inertial_cylinder mass="0.1" length="0.01" radius="0.045">
+        <xacro:inertial_cylinder mass="0.25" length="0.01" radius="0.045">
             <origin xyz="0 0 0" rpy="0 0 0"/>
         </xacro:inertial_cylinder>
@@ -83,7 +68,4 @@
         <axis xyz="0.0 0.0 1.0"/>
     </joint>
-    <!-- <gazebo reference="front_left_wheel_link">
-        <material>Gazebo/Blue</material>
-    </gazebo> -->
     <!-- front right wheel -->
     <link name="front_right_wheel_joint_link">
@@ -105,15 +87,13 @@
             <origin xyz="0.0 0.0 -0.005" rpy="1.57 0.0 0.0"/>
             <geometry>
-                <mesh filename="file://$(find ${description_package})/meshes/limo_wheel.dae"/>
+                <mesh filename="file://$(find ${description_package})/meshes/limo_optimal_wheels.dae"/>
             </geometry>
-            <!-- <material name="blue"/> -->
         </visual>
         <collision>
-            <!-- <origin xyz="0.0 0.0 0.0" rpy="0.0 0.0 0.0"/> -->
             <geometry>
                 <cylinder radius="0.045" length="0.01"/>
             </geometry>
         </collision>
-        <xacro:inertial_cylinder mass="0.1" length="0.01" radius="0.045">
+        <xacro:inertial_cylinder mass="0.25" length="0.01" radius="0.045">
             <origin xyz="0 0 0" rpy="0 0 0"/>
         </xacro:inertial_cylinder>
@@ -125,7 +105,4 @@
         <axis xyz="0.0 0.0 -1.0"/>
     </joint>
-    <!-- <gazebo reference="front_right_wheel_link">
-        <material>Gazebo/Blue</material>
-    </gazebo> -->
     <!-- back left wheel -->
     <joint name="back_left_wheel" type="continuous">
@@ -139,21 +116,15 @@
             <origin xyz="0 0 -0.005" rpy="1.57 0 0"/>
             <geometry>
-                <mesh filename="file://$(find ${description_package})/meshes/limo_wheel.dae"/>
+                <mesh filename="file://$(find ${description_package})/meshes/limo_optimal_wheels.dae"/>
             </geometry>
-            <!-- <material name="black"/> -->
         </visual>
-        <collision>
-            <!-- <origin xyz="0.0 0.0 0.0" rpy="0.0 0.0 0.0"/> -->
-            <geometry>
+        <collision>            <geometry>
                 <cylinder radius="0.045" length="0.01"/>
             </geometry>
         </collision>
-        <xacro:inertial_cylinder mass="0.1" length="0.01" radius="0.045">
+        <xacro:inertial_cylinder mass="0.25" length="0.01" radius="0.045">
             <origin xyz="0 0 0" rpy="0 0 0"/>
         </xacro:inertial_cylinder>
     </link>
-    <!-- <gazebo reference="back_left_wheel_link">
-        <material>Gazebo/Black</material>
-    </gazebo> -->
     <!-- back right wheel -->
     <joint name="back_right_wheel" type="continuous">
@@ -168,20 +139,15 @@
             <origin xyz="0 0 -0.005" rpy="1.57 0 0"/>
             <geometry>
-                <mesh filename="file://$(find ${description_package})/meshes/limo_wheel.dae"/>
+                <mesh filename="file://$(find ${description_package})/meshes/limo_optimal_wheels.dae"/>
             </geometry>
-            <!-- <material name="black"/> -->
         </visual>
         <collision>
-            <!-- <origin xyz="0.0 0.0 0.0" rpy="0.0 0.0 0.0"/> -->
             <geometry>
                 <cylinder radius="0.045" length="0.01"/>
             </geometry>
         </collision>
-        <xacro:inertial_cylinder mass="0.1" length="0.01" radius="0.045">
+        <xacro:inertial_cylinder mass="0.25" length="0.01" radius="0.045">
             <origin xyz="0 0 0" rpy="0 0 0"/>
         </xacro:inertial_cylinder>
     </link>
-    <!-- <gazebo reference="back_right_wheel_link">
-        <material>Gazebo/Black</material>
-    </gazebo> -->
 </robot>

File: src/robot_description/description/robot-main.xacro (robot description, xacro)
@@ -5,6 +5,6 @@
     <xacro:include filename="$(find robot_description)/description/limo_core.urdf.xacro"/>
     <xacro:include filename="$(find robot_description)/description/gazebo_control.xacro"/>
-    <!-- <xacro:include filename="$(find robot_description)/description/camera.xacro"/> -->
+    <xacro:include filename="$(find robot_description)/description/camera.xacro"/>
     <!-- <xacro:include filename="$(find robot_description)/description/lidar.xacro"/> -->
-    <!-- <xacro:include filename="$(find robot_description)/description/imu.xacro"/> -->
+    <xacro:include filename="$(find robot_description)/description/imu.xacro"/>
 </robot>

Commit message: Move pkg to folder

File: src/robot_description/description/camera.xacro (robot description, xacro)
@@ -2,5 +2,5 @@
 <robot xmlns:xacro="http://www.ros.org/wiki/xacro" >
     <joint name="camera_joint" type="fixed">
-        <parent link="chassis"/>
+        <parent link="base_link"/>
         <child link="camera_link"/>
         <origin xyz="0.190 0.0 0.135" rpy="0 0 0"/>

File: src/robot_description/description/imu.xacro (robot description, xacro)
@@ -2,5 +2,5 @@
 <robot xmlns:xacro="http://www.ros.org/wiki/xacro" >
     <joint name="imu_joint" type="fixed">
-        <parent link="chassis"/>
+        <parent link="base_link"/>
         <child link="imu_link"/>
         <origin xyz="0.05 0.0 0.07" rpy="0 0 0"/>

Commit message: Readme update lab1.1 v.1

File: src/robot_description/description/camera.xacro (robot description, xacro)
@@ -4,5 +4,5 @@
         <parent link="base_link"/>
         <child link="camera_link"/>
-        <origin xyz="0.190 0.0 0.135" rpy="0 0 0"/>
+        <origin xyz="0.09 0.0 0.13" rpy="0 0 0"/>
     </joint>
     <link name="camera_link">

File: src/robot_description/description/imu.xacro (robot description, xacro)
@@ -4,21 +4,13 @@
         <parent link="base_link"/>
         <child link="imu_link"/>
-        <origin xyz="0.05 0.0 0.07" rpy="0 0 0"/>
+        <origin xyz="0.09 0.0 0.13" rpy="0 0 0"/>
     </joint>
     <link name="imu_link">
         <visual>
             <geometry>
-                <cylinder radius="0.05" length="0.04"/>
+                <box size="0.010 0.03 0.03"/>
             </geometry>
             <material name="red"/>
         </visual>
-        <collision>
-            <geometry>
-                <cylinder radius="0.05" length="0.04"/>
-            </geometry>
-        </collision>
-        <xacro:inertial_cylinder mass="0.1" length="0.04" radius="0.05">
-            <origin xyz="0 0 0" rpy="0 0 0"/>
-        </xacro:inertial_cylinder>
     </link>
     <gazebo reference="imu_link">
